File: circuito/ControleMix.sch (KiCad schematic (older format))
At the start: 32 parts, among them J1 AIN0, J10 OUT1, J11 AIN5, J12 OUT2, J13 AIN6, J14 OUT3, J15 AIN7, J16 OUT4, J17 AIN8, J18 AIN9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

Commit message: code
Changed lines of the file:
@@
 PB3
 Text Label 4950 5900 0    50   ~ 0
-PB15
+PA15
 Wire Wire Line
 	4950 5900 4650 5900
@@
 	3000 2650 3000 2550
 Text Label 10250 2750 0    50   ~ 0
-PB15
+PA15
 Text Label 10250 2650 0    50   ~ 0
 PB3
